Commit message: ft[updates]: Working examples for boxer, panda and point robot.

File: examples/panda_fk.urdf (robot description, URDF)
Before this commit: robot panda, 9 links, 8 joints
Links:
- added link panda_link8
Joints:
- added joint panda_joint8: type fixed, parent panda_link7, child panda_link8, origin xyz=0 0 0.10 rpy=0 0 0, axis 0 0 1
